File: SharkBait_328/SharkBait_328.brd (EAGLE design)
At the start: 42 x 94 mm, 29 parts, among them J1 BC501SM-TR, U1 DS3231M+, U2 328P

Commit message: routing v1
Routing:
- net GND: track 0.00 -> 204.7 mm, vias 0 -> 4
- net 5V: track 0.00 -> 136.8 mm, vias 0 -> 2
- net 3V3: track 0.00 -> 62.6 mm, vias 0 -> 4
- net D6: track 0.00 -> 49.3 mm
- net SCL: track 0.00 -> 44.1 mm, vias 0 -> 1
- net N$10: track 0.00 -> 42.5 mm, vias 0 -> 2
- net N$2: track 0.00 -> 38.7 mm, vias 0 -> 2
- net N$4: track 0.00 -> 35.8 mm
- net N$1: track 0.00 -> 34.0 mm
- net A2: track 0.00 -> 33.7 mm
- net VIN: track 0.00 -> 33.3 mm
- net N$8: track 0.00 -> 29.3 mm, vias 0 -> 1
- net D4-POWSENS: track 0.00 -> 28.5 mm
- net A1: track 0.00 -> 28.1 mm
- net A0: track 0.00 -> 25.4 mm
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